File: sensors/imu/aspirin/v2.1/aspirin.sch (EAGLE design)
At the start: 23 parts, among them IC1 LP2992, IC2 MS5611, IC3 >4KBIT SERIAL EEPROM HALF PRO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, U1 HMC5883, U2 MPU-6000

Commit message: Minor final fixes before going into assembly.
Parts:
- C1, IC2: DNP (none) -> T
- C13: PARTNO cap-cer-0603-4n7 -> cap-cer-0603-4u7
- C5: PARTNO cap-cer-0402-4n7 -> cap-cer-0603-4u7
Other:
- note removed: "(C) 2011 Joby Robotics <info@jobyrobotics.com>"
Changed lines of the file:
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@@
 </part>
 <part name="C5" library="pel_dipol_comp" deviceset="CAPACITOR" device="-0603" value="4.7uF/10V/Low ESR">
-<attribute name="PARTNO" value="cap-cer-0402-4n7"/>
+<attribute name="PARTNO" value="cap-cer-0603-4u7"/>
 </part>
 <part name="GND1" library="supply1" deviceset="GND" device=""/>
@@
 </part>
 <part name="C13" library="pel_dipol_comp" deviceset="CAPACITOR" device="-0603" value="4.7uF/10V/Low ESR">
-<attribute name="PARTNO" value="cap-cer-0603-4n7"/>
+<attribute name="PARTNO" value="cap-cer-0603-4u7"/>
 </part>
 <part name="GND10" library="supply1" deviceset="GND" device=""/>
@@
 </part>
 <part name="IC2" library="aspirin" deviceset="MS5611" device="">
+<attribute name="DNP" value="T"/>
 <attribute name="PARTNO" value="sensr-qfn-8-baro"/>
 </part>
 <part name="C1" library="pel_dipol_comp" deviceset="CAPACITOR" device="-0402" value="100n">
+<attribute name="DNP" value="T"/>
 <attribute name="PARTNO" value="cap-cer-0402-100n"/>
 </part>
@@
 <text x="187.96" y="25.4" size="1.27" layer="97">License: CC-BY-SA 3.0</text>
 <text x="210.82" y="25.4" size="1.27" layer="97">http://creativecommons.org/licenses/by-sa/3.0</text>
-<text x="168.91" y="30.48" size="1.27" layer="97">(C) 2010-2011 Piotr Esden-Tempski &lt;piotr@esden.net&gt;</text>
+<text x="217.17" y="30.48" size="1.27" layer="97">(C) 2010-2011 Piotr Esden-Tempski &lt;piotr@esden.net&gt;</text>
 <text x="168.91" y="33.02" size="1.27" layer="97">(C) 2010-2011 Antoine Drouin &lt;poinix@gmail.com&gt;</text>
 <text x="217.17" y="33.02" size="1.27" layer="97">(C) 2011 Richard Hatano &lt;rhatano@jobyenergy.com&gt;</text>
-<text x="217.17" y="30.48" size="1.27" layer="97">(C) 2011 Joby Robotics &lt;info@jobyrobotics.com&gt;</text>
-<text x="168.91" y="27.94" size="1.27" layer="97">(C) 2011 Transition Robotics &lt;info@transition-robotics.com&gt;</text>
+<text x="168.91" y="30.48" size="1.27" layer="97">(C) 2011 Transition Robotics &lt;info@transition-robotics.com&gt;</text>
 </plain>
 <instances>
@@
 </instance>
 <instance part="C5" gate="G$1" x="60.96" y="152.4">
-<attribute name="PARTNO" value="cap-cer-0603-4u7" x="60.96" y="152.4" size="1.778" layer="96" display="off"/>
+<attribute name="PARTNO" value="cap-cer-0603-4n7" x="60.96" y="152.4" size="1.778" layer="96" display="off"/>
 </instance>
 <instance part="GND1" gate="1" x="162.56" y="104.14" rot="MR0"/>
@@
 <attribute name="NAME" x="219.964" y="142.621" size="1.778" layer="95"/>
 <attribute name="VALUE" x="230.759" y="131.064" size="1.778" layer="96" rot="R90"/>
-<attribute name="PARTNO" value="cap-cer-0603-4u7" x="226.06" y="142.24" size="1.778" layer="96" display="off"/>
+<attribute name="PARTNO" value="cap-cer-0603-4n7" x="226.06" y="142.24" size="1.778" layer="96" display="off"/>
 </instance>
 <instance part="GND10" gate="1" x="226.06" y="121.92" rot="MR0"/>
@@
 <attribute name="DNP" x="152.4" y="83.82" size="1.778" layer="96" display="both"/>
 </instance>
-<instance part="IC2" gate="G$1" x="38.1" y="96.52">
+<instance part="IC2" gate="G$1" x="38.1" y="96.52" smashed="yes">
 <attribute name="PARTNO" value="sensr-qfn-8-baro" x="38.1" y="96.52" size="1.778" layer="96" display="off"/>
+<attribute name="DNP" x="38.1" y="86.36" size="1.778" layer="96" display="both"/>
+<attribute name="NAME" x="27.94" y="106.68" size="1.27" layer="95" rot="MR180"/>
+<attribute name="VALUE" x="27.94" y="86.36" size="1.27" layer="96"/>
 </instance>
 <instance part="C1" gate="G$1" x="15.24" y="91.44" rot="MR0">
 <attribute name="PARTNO" value="cap-cer-0402-100n" x="15.24" y="91.44" size="1.778" layer="96" display="off"/>
+<attribute name="DNP" x="7.62" y="93.98" size="1.778" layer="96" rot="MR270" display="both"/>
 </instance>
 <instance part="GND4" gate="1" x="20.32" y="78.74" rot="MR0"/>

Commit message: Fixed the corner pin intended for GYRO_CS to be disconnected from ground and labeled RESV on the pcb.
Connections:
- net GND: no longer ASP1.GND@3
Changed lines of the file:
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@@
 <?xml version="1.0" encoding="utf-8"?>
 <!DOCTYPE eagle SYSTEM "eagle.dtd">
-<eagle version="6.1">
+<eagle version="6.2">
 <drawing>
 <settings>
@@
 <wire x1="73.66" y1="50.8" x2="71.12" y2="50.8" width="0.1524" layer="91"/>
 <wire x1="109.22" y1="66.04" x2="111.76" y2="66.04" width="0.1524" layer="91"/>
-<wire x1="111.76" y1="66.04" x2="111.76" y2="50.8" width="0.1524" layer="91"/>
-<wire x1="111.76" y1="50.8" x2="111.76" y2="45.72" width="0.1524" layer="91"/>
+<wire x1="111.76" y1="66.04" x2="111.76" y2="45.72" width="0.1524" layer="91"/>
 <wire x1="111.76" y1="45.72" x2="91.44" y2="45.72" width="0.1524" layer="91"/>
 <wire x1="91.44" y1="45.72" x2="71.12" y2="45.72" width="0.1524" layer="91"/>
 <wire x1="71.12" y1="45.72" x2="71.12" y2="50.8" width="0.1524" layer="91"/>
-<wire x1="109.22" y1="50.8" x2="111.76" y2="50.8" width="0.1524" layer="91"/>
 <wire x1="91.44" y1="45.72" x2="91.44" y2="43.18" width="0.1524" layer="91"/>
 <junction x="71.12" y="50.8"/>
-<junction x="111.76" y="50.8"/>
 <junction x="91.44" y="45.72"/>
 <pinref part="ASP1" gate="G$1" pin="GND@1"/>
 <pinref part="ASP1" gate="G$1" pin="GND@2"/>
 <pinref part="ASP1" gate="G$1" pin="GND@4"/>
-<pinref part="ASP1" gate="G$1" pin="GND@3"/>
 <pinref part="GND3" gate="1" pin="GND"/>
 </segment>
