File: controller/lisa_m/v2.1/lisa_m.sch (EAGLE design)
At the start: 119 parts, among them IC9 LP2992 5V, J1 CONN_3-1, J2 CONN_3-1, J3 CONN_3-1, J4 CONN_3-1, J5 CONN_3-1, J6 CONN_3-1, J7 CONN_3-1, J8 CONN_3-1, Q1 12Mhz, U1 MCP2551SN, U2 STM32-C-64, U3 BMP085

Commit message: Updated V2.1 Lisa/M(X) hardware to the final production version.
Parts:
- removed C8: 100n, pel_dipol_comp:CAPACITOR-0402
- removed CON_ANALOG2: (no value), pel_molex:CONN_6-1-53398
- removed IMU: ASPIRIN, joby_robotics:ASPIRIN
- removed J1, J2, J3, J4, J5, J6, J7, J8: CONN_3-1, pel_misc:CONN_3-1
- removed JP4, JP5: 0/DNP, pel_jumpers:SQ_JMP-0402
- removed LED6, LED7, LED8, LED9: BLU, pel_dipol_comp:LED-0402
- removed R32, R35, R36: 80R, pel_dipol_comp:RESISTOR-0402
- removed U$1: TR-LOGO, quadshot:TR-LOGO
- removed U3: BMP085, omc:BMP085
- added C101, C108, C110, C112: 100n, pel_dipol_comp:CAPACITOR-0402
- added C104: 2u2, pel_dipol_comp:CAPACITOR-0603
- added C105, C113: 4u7, pel_dipol_comp:CAPACITOR-0603
- added C106: 10n, pel_dipol_comp:CAPACITOR-0402
- added C109: 2n2, pel_dipol_comp:CAPACITOR-0402
- added C114: 220n, pel_dipol_comp:CAPACITOR-0603
- added IC101: LP2992, v-reg-micrel:MIC5219BM5
- added IC102: MS5611, aspirin:MS5611
- added L101: L, pel_dipol_comp:INDUCTOR-0402
- added LEDVIN: GRN, pel_dipol_comp:LED-0402
- added PH1, PH2, PH3, PH4: PH2X3, pel_hdr:PH2X3
- added R11, R9: 2k2, pel_dipol_comp:RESISTOR-0402
- added SW1: MICROTACT_GND, paparazzi:MICROTACT_GND
- added U102: MPU-6000, aspirin:MPU-6000
- added U103: HMC5883L, aspirin:HMC5883L
- C1, C9: device pel_dipol_comp:CAPACITOR-0805 -> pel_dipol_comp:CAPACITOR-0603; PARTNO C2012Y5V1C475Z/1.25 -> cap-cer-0603-4u7
- C10, C11, C12, C14, C15, C2, C27, C38, C5, C7: PARTNO LMK105BJ104KV-F -> cap-cer-0402-100n
- C13, C31: PARTNO CC0402KRX7R9BB103 -> cap-cer-0402-10n
- C26, C3, C36: device pel_dipol_comp:CAPACITOR-0603 -> pel_dipol_comp:CAPACITOR-0402; PARTNO C0603C104K5RACTU -> cap-cer-0402-100n
- C28: device pel_dipol_comp:CAPACITOR-POL-0603 -> pel_dipol_comp:CAPACITOR-0603; PARTNO F981E105MMA -> cap-cer-0603-1u
- C35: PARTNO CC0402KRX7R9BB471 -> cap-cer-0402-470p
- C37, C39: PARTNO T491B226M016AT -> cap-tan-B-22u-16v
- C4, C6: value 30p -> 10p; PARTNO C1005C0G1H300J -> cap-cer-0402-10p
- C42: PARTNO C0603C472K5RACTU -> cap-cer-0603-4n7
- CON_ANALOG1, CON_UART1/5: PARTNO 53398-0671 -> conn-picoblade-smd-0.05in-6-vert
- CON_CAN/I2C1: device pel_molex:CONN_7-1-53261 -> pel_molex:CONN_7-1-53398; PARTNO 53398-0771 -> conn-picoblade-smd-0.05in-7-vert
- CON_GPIO, CON_I2C2, CON_UART2, CON_UART3: PARTNO 53398-0471 -> conn-picoblade-smd-0.05in-4-vert
- CON_SPI: PARTNO 53398-0771 -> conn-picoblade-smd-0.05in-7-vert
- CON_USB: DNP (none) -> T; PARTNO 53047-0410 -> conn-picoblade-th-0.05in-4-vert
- CON_USB_MICRO: PARTNO ZX62-B-5PA(11) -> conn-smd-usb-micro-b
- D3: device diode:DIODE-MICROMELF-R -> pel_dipol_comp:DIODE-0603; PARTNO RB160SS-40T2R -> diode-schottky-0603
- IC9: PARTNO LP2992IM5-5.0/NOPB -> vreg-sot-23-5-5v
- JP1, JP12, JP13, JP2, JP3, JP6, JP7, JP8, JP9, R56: PARTNO RC0402JR-070RL -> res-0402-0
- JP10, JP11: PARTNO RC0603JR-070RL -> res-0603-0
- JTAG: PARTNO FTSH-105-01-F-DV-K-P-TR -> conn-smd-0.05in-5-2
- L1: value INDUCTOR-0603 -> L; device res_cap:INDUCTOR-0603 -> pel_dipol_comp:INDUCTOR-0402; PARTNO MMZ1608B601C -> ferrite-0402-600
- LED1: PARTNO SML-P11UTT86 -> led-0402-red
- LED2: value BLU -> ORG; PARTNO SMLP12BC7TT86 -> led-0402-org
- LED3: value BLU -> GRN; DNP T -> (none); PARTNO SMLP12BC7TT86 -> led-0402-grn
- LED4: value ORG -> YEL; PARTNO SML-P11DTT86 -> led-0402-yel
- LED5: value BLU -> RED; DNP T -> (none); PARTNO SMLP12BC7TT86 -> led-0402-grn
- LT_I2C2: PARTNO PCA9306DP,118 -> ic-tssop8-level-trans
- Q1: PARTNO ABM8-12.000MHZ-B2-T -> xtal-abm8-12mhz
- R1: value 22R -> 10k; PARTNO ERJ-2GEJ220X -> res-0402-10k
- R10, R12, R37, R38: value 80R -> 300; PARTNO RMCF0402JT470R -> res-0402-300
- R17, R7: PARTNO RMCF0402JT10K0 -> res-0402-10k
- R18: value 2k -> 2k2; PARTNO RMCF0402FT2K00 -> res-0402-2k2
- R2: value 22R -> 2k2; PARTNO ERJ-2GEJ220X -> res-0402-2k2
- R23: value 2k -> 2k2; PARTNO RMCF0402JT1K50 -> res-0402-2k2
- R24, R26, R29, R3, R30, R6: value 2k7 -> 10k; PARTNO RMCF0402JT2K70 -> res-0402-10k
- R25: PARTNO RC0402JR-07200KL -> res-0402-200k
- R27, R28, R31, R39, R40, R41, R42, R45: PARTNO RC0402JR-07100RL -> res-0402-100
- R33, R34, R4, R5: value 2k7 -> 2k2; PARTNO RMCF0402JT2K70 -> res-0402-2k2
- R43, R44: value 1k5 -> 2k2; PARTNO RMCF0402JT1K50 -> res-0402-2k2
- R55: PARTNO RC0603JR-070RL -> res-0402-10k
- R58, R59: PARTNO ERJ-2RKF60R4X -> res-0402-60.4
- R60, R61: PARTNO RMCF0402JT4K70 -> res-0402-4k7
- R8: value 300R -> 300; PARTNO RMCF0402JT470R -> res-0402-300
- U1: PARTNO MCP2551-I/SN -> ic-so8-can
- U2: PARTNO STM32F105RCT6 -> ic-mcu-stm32f415rgt6
- VREG1: PARTNO MIC5209-3.3YM -> vreg-so8-3v3
Connections:
- removed net ADC_4: CON_ANALOG2.4, LED7.C, U2.PC5-ADC15ETH_(R)MII_RXD1
- removed net ADC_6: CON_ANALOG2.5, LED8.C, U2.PC2-ADC12/ETH_MII_TXD2
- removed net FT_USB_DM: CON_USB.2, CON_USB_MICRO.2, R1.1
- removed net FT_USB_DP: CON_USB.3, CON_USB_MICRO.3, R2.1
- removed net IMU_ACC_CS: IMU.ACC_CS, U2.PB12-SPI2NSS/I2S2WS/I2C2SMBA/USART3CK/TIM1BKIN/CAN2RX/ETH_(R)MII_TXD0
- removed net IMU_ACC_DRDY: IMU.ACC_DRDY, U2.PB2/BOOT1
- removed net IMU_GYRO_DRDY: IMU.GYRO_DRDY, U2.PC14-OSC32_IN
- removed net IMU_GYRO_SS: IMU.GND3, U2.PC13-TAMPER-RTC
- removed net IMU_MAG_DRDY: IMU.MAG_DRDY, R29.2, U2.PB5-I2C1SMBA/SPI3MOSI/ETH_(R)MII_PPS_OUT/I2S3SD-TIM3CH2/SPI1MOSI/CAN2RX
- removed net JTAG_TRST: CON_GPIO.4, LED1.C, U2.PB4/JNTRST-SPI3MISO-TIM3CH1/SPI1MISO
- removed net N$11: LED6.A, R36.1
- removed net N$9: LED5.A, R35.1
- removed net U2_POW: CON_UART2.2, JP4.2, JP5.2, R26.1
- new net BARO_+3V3: C101.1, IC102.VDD, L101.1
- new net BIND_BUT: R11.2, SW1.2, U2.PB2/BOOT1
- new net IMU+3V3: C105.1, C108.1, C112.1, IC101.OUT, L101.2, U102.VDD, U103.S1, U103.VDD, U103.VDDIO
- new net IMU_BARO_CS: IC102.!CSB@1, IC102.!CSB@2, U2.PC13-TAMPER-RTC
- new net IMU_MAG_INT: U103.DRDY, U2.PC14-OSC32_IN
- new net IMU_MPU_CS: U102.!CS, U2.PB12-SPI2NSS/I2S2WS/I2C2SMBA/USART3CK/TIM1BKIN/CAN2RX/ETH_(R)MII_TXD0
- new net IMU_MPU_INT: R29.2, U102.INT, U2.PB5-I2C1SMBA/SPI3MOSI/ETH_(R)MII_PPS_OUT/I2S3SD-TIM3CH2/SPI1MOSI/CAN2RX
- new net LED3: LED3.C, U2.PC2-ADC12/ETH_MII_TXD2
- new net LED4: LED4.C, U2.PC5-ADC15ETH_(R)MII_RXD1
- new net LED5: LED5.C, U2.PC15-OSC32_OUT
- new net N$19: C106.2, IC101.ADJ
- new net N$2: C109.1, U102.CPOUT
- new net N$3: C110.1, U102.REGOUT
- new net N$34: C114.2, U103.SETP
- new net N$48: C114.1, U103.SETC
- new net SCL: R9.1, U102.AUX_CL, U103.SCL
- new net SDA: R2.1, U102.AUX_DA, U103.SDA
- net +3V3: now also CON_UART2.2, R11.1, R2.2, R26.1, R9.2; no longer C8.2, CON_ANALOG2.2, JP5.1, R32.2, R35.2, R36.2, U3.VDDA, U3.VDDD
- net +5V: no longer CON_ANALOG2.3
- net ADC_1: no longer LED3.C
- net ADC_2: no longer LED5.C
- net ADC_3: no longer LED6.C
- net BARO_DRDY: no longer U3.EOC
- net BOOT0: no longer CON_ANALOG2.6
- net GND: now also C101.2, C104.2, C105.2, C106.1, C108.2, C109.2, C110.2, C112.2, C113.2, C28.2, IC101.GND, IC102.GND, IC102.PS, LEDVIN.C, PH1A.3, PH1B.3, PH2A.3, PH2B.3, PH3A.3, PH3B.3, PH4A.3, PH4B.3, R1.2, SW1.1, SW1.GND, U102.CLKIN, U102.FSYNC, U102.GND, U103.GND, U103.GND2; no longer C28.-, C8.1, CON_ANALOG2.1, IMU.GND1, IMU.GND2, IMU.GND4, J1.1, J2.1, J3.1, J4.1, J5.1, J6.1, J7.1, J8.1, LED4.C, U3.GND
- net I2C2_SCL: no longer IMU.SCL, U3.SCL
- net I2C2_SDA: no longer IMU.SDA, U3.SDA
- net IMU_SPI_MISO: now also IC102.SDO, U102.AD0/SDO; no longer IMU.MISO
- net IMU_SPI_MOSI: now also IC102.SDI/SDA, U102.SDA/SDI; no longer IMU.MOSI
- net IMU_SPI_SCK: now also IC102.SCLK, U102.SCL/SCLK; no longer IMU.SCK
- net LED1: now also LED1.C; no longer LED2.C
- net LED2: now also CON_GPIO.4, LED2.C, U2.PB4/JNTRST-SPI3MISO-TIM3CH1/SPI1MISO; no longer LED9.C, U2.PC15-OSC32_OUT
- net N$10: now also LED2.A; no longer LED1.A
- net N$12: now also LEDVIN.A; no longer LED4.A
- net N$13: now also LED5.A; no longer LED9.A
- net N$14: now also LED4.A; no longer LED7.A
- net N$15: now also LED3.A; no longer LED8.A
- net N$4: now also LED1.A; no longer LED2.A
- net N$5: now also C113.1, U103.C1; no longer LED3.A, R32.1
- net S1: now also PH1A.1; no longer J1.3
- net S2: now also PH1B.1; no longer J2.3
- net S3: now also PH2A.1; no longer J3.3
- net S4: now also PH2B.1; no longer J4.3
- net S5: now also PH3A.1; no longer J5.3
- net S6: now also PH3B.1; no longer J6.3
- net S7: now also PH4A.1; no longer J7.3
- net S8: now also PH4B.1; no longer J8.3
- net SERVO_BUS: now also PH1A.2, PH1B.2, PH2A.2, PH2B.2, PH3A.2, PH3B.2, PH4A.2, PH4B.2; no longer J1.2, J2.2, J3.2, J4.2, J5.2, J6.2, J7.2, J8.2
- net USB_DM: now also CON_USB.2, CON_USB_MICRO.2; no longer R1.2
- net USB_DP: now also CON_USB.3, CON_USB_MICRO.3; no longer R2.2
- net USB_VBUS: now also R1.1
- net VDDA: now also C28.1; no longer C28.+
- net V_IN: now also C104.1, IC101.EN, IC101.IN; no longer IMU.VCC, JP4.1
Other:
- note added: "(C) 2010-2014 Piotr Esden-Tempski <piotr@esden.net>"
- note added: "1BitSquared LLC"
- note added: "3V3 DIGITAL"
- note added: "Accelerometer & Gyroscope"
- note added: "Bind Button"
- note added: "Lisa/M(X) V2.1"
- note added: "Magnetometer"
- note added: "Presure"
- note added: "R3"
- note added: "SWCLK"
- note added: "SWDIO"
- note added: "TRACESWO"
- note removed: "(128/20)"
- note removed: "(512/64)"
- note removed: "(C) 2010-2011 Piotr Esden-Tempski <piotr@esden.net>"
- note removed: "- address encoding by solder jumpers ?"
- note removed: "-2*5 pins with GND, 5V, 3V3, IO1, IO2 ( PWM in/out, adc, i2c if possible)"
- note removed: "-8 reset power supervisor"
- note removed: "-Medium density family"
- note removed: "1"
- note removed: "1 optional max ( 232/485 ), 1 optional 5V ( spare channel of servo driver)"
- note removed: "10 pins Piotr :)"
- note removed: "11.22$"
- note removed: "2"
- note removed: "2 * 4 pins molex 2.54"
- note removed: "2 * 5 pins picoblade"
- note removed: "2 * 7 pins picoblade"
- note removed: "2 pins MOLEX 2.54mm"
- note removed: "30$"
- note removed: "4"
- note removed: "48 pin QFP or 36 pin QFN ? ( QFP is nicer to service )"
- note removed: "4pin picoblade/ mini USB ?"
- note removed: "50$"
- note removed: "5V PHY driver"
- note removed: "5V rail for CAN, 3V3 rail for the rest"
- note removed: "5V shifting for signal"
- note removed: "6"
- note removed: "6 * 3 pins MOLEX 2.54mm"
- note removed: "6 pins picoblade"
- note removed: "7.1$"
- note removed: "8"
- note removed: "8 pins picoblade"
- note removed: "?? 2 pins picoblade"
- note removed: "ADCs"
- note removed: "ANALOG2"
- note removed: "Add connector for no aspirin"
- note removed: "Affordable"
- note removed: "BARO"
- note removed: "Budget"
- note removed: "CAN"
- note removed: "CONNECTOR"
- note removed: "DRIVER"
- note removed: "FIXME"
- note removed: "FLASHING:"
- note removed: "FUNCTION"
- note removed: "GPIOs"
- note removed: "Goals"
- note removed: "I2C"
- note removed: "IMU"
- note removed: "IOs:"
- note removed: "JTAG on 10 pin 1.25 mm headers"
- note removed: "LEDs"
- note removed: "LEVEL CONV"
- note removed: "MAX"
- note removed: "MCU direct"
- note removed: "MCU:"
- note removed: "MIN"
- note removed: "Misc"
- note removed: "N/A"
- note removed: "PCA9306 : 3V3, 5V, external level"
- note removed: "Rugged"
- note removed: "STM32F103RB"
- note removed: "STM32F103RE"
- note removed: "SUPPLY"
- note removed: "Servos"
- note removed: "Specifications"
- note removed: "Supply:"
- note removed: "TOTAL"
- note removed: "UARTs"
- note removed: "a couple of resistor bridges"
- note removed: "analog domain - separate rail ( I vote no separate regulator for analog )?"
- note removed: "crystal to save cost ( not external oscillator )"
- note removed: "easy to manufacture"
- note removed: "easy to service"
- note removed: "fixed via aspirin-connector dummy bd"
- note removed: "flash/run button switch"
- note removed: "for flashing through bootloader"
- note removed: "http://transition-robotics.com"
- note removed: "input voltage : 6 cells - 25V"
- note removed: "linear reg ?"
- note removed: "populated only on dev boards"
- note removed: "power switch"
- note removed: "serial flashing on prod boards"
